File: DA14531MOD-Breakout/DA14531MOD-Breakout.sch (KiCad schematic (older format))
At the start: 3 parts, among them J1 Conn_01x07, J2 Conn_01x07, U1 DA14531MOD-00F01002

Commit message: finetuning
Connections:
- net J10_P02_SWDCLK: now also J2.6 (Pin_6); no longer J1.7 (Pin_7)
- net J8_P0_11: now also J1.7 (Pin_7); no longer J1.5 (Pin_5)
- net J9_P010_SWDIO: now also J2.7 (Pin_7); no longer J1.6 (Pin_6)
- net VDD: now also J1.5 (Pin_5), J1.6 (Pin_6); no longer J2.6 (Pin_6), J2.7 (Pin_7)
Changed lines of the file:
@@
 Text Label 4350 3400 2    50   ~ 0
 J5_P0_6
-Text Label 2125 3250 0    50   ~ 0
+Text Label 2125 3050 0    50   ~ 0
 J8_P0_11
 Text Label 5950 3300 0    50   ~ 0
@@
 Text Label 7975 3400 2    50   ~ 0
 J12_P00_RST
-Text Label 6925 4025 0    50   ~ 0
+Text Label 7975 3500 2    50   ~ 0
 J10_P02_SWDCLK
 $Comp
@@
 Text Label 7975 3300 2    50   ~ 0
 J16_P0_7
-Text Label 2125 3150 0    50   ~ 0
+Text Label 2675 2700 0    50   ~ 0
 J9_P010_SWDIO
 $Comp
@@
 $EndComp
 $Comp
-L power:VDD #PWR0102
-U 1 1 602F9100
-P 7975 3600
-F 0 "#PWR0102" H 7975 3450 50  0001 C CNN
-F 1 "VDD" V 7990 3728 50  0000 L CNN
-F 2 "" H 7975 3600 50  0001 C CNN
-F 3 "" H 7975 3600 50  0001 C CNN
-	1    7975 3600
-	0    -1   -1   0
-$EndComp
-$Comp
 L power:PWR_FLAG #FLG0101
 U 1 1 602FAD7C
@@
 Connection ~ 5950 3700
 $Comp
-L power:VDD #PWR01
-U 1 1 602F288D
-P 7975 3500
-F 0 "#PWR01" H 7975 3350 50  0001 C CNN
-F 1 "VDD" V 7990 3628 50  0000 L CNN
-F 2 "" H 7975 3500 50  0001 C CNN
-F 3 "" H 7975 3500 50  0001 C CNN
-	1    7975 3500
-	0    -1   -1   0
-$EndComp
-Text Label 2125 3050 0    50   ~ 0
-J10_P02_SWDCLK
-$Comp
-L power:GND #PWR?
+L power:GND #PWR0102
 U 1 1 60305DB2
 P 2125 3450
-F 0 "#PWR?" H 2125 3200 50  0001 C CNN
+F 0 "#PWR0102" H 2125 3200 50  0001 C CNN
 F 1 "GND" V 2130 3322 50  0000 R CNN
 F 2 "" H 2125 3450 50  0001 C CNN
@@
 	0    -1   -1   0
 $EndComp
+$Comp
+L power:VDD #PWR0103
+U 1 1 602E62E8
+P 2125 3250
+F 0 "#PWR0103" H 2125 3100 50  0001 C CNN
+F 1 "VDD" H 2140 3423 50  0000 C CNN
+F 2 "" H 2125 3250 50  0001 C CNN
+F 3 "" H 2125 3250 50  0001 C CNN
+	1    2125 3250
+	0    1    1    0
+$EndComp
+$Comp
+L power:VDD #PWR0104
+U 1 1 602E7148
+P 2125 3150
+F 0 "#PWR0104" H 2125 3000 50  0001 C CNN
+F 1 "VDD" H 2140 3323 50  0000 C CNN
+F 2 "" H 2125 3150 50  0001 C CNN
+F 3 "" H 2125 3150 50  0001 C CNN
+	1    2125 3150
+	0    1    1    0
+$EndComp
+Text Label 7975 3600 2    50   ~ 0
+J9_P010_SWDIO
 $EndSCHEMATC
